Commit message: Separeted file creation for colors

File: src/MineMapper_bringup/URDF/MineMapper.urdf.xacro (robot description, xacro)
@@ -1,4 +1,7 @@
 <?xml version="1.0"?>
 <robot name="MineMapper" xmlns:xacro="http://www.ros.org.wiki/xacro">
+    <!-- INCLUDES -->
+    <xacro:include filename="commom_properties.xacro"/>
+    <!-- PROPERTIES -->
     <xacro:property name="base_length" value="0.6"/>
     <xacro:property name="base_width" value="0.4"/>
@@ -6,10 +9,4 @@
     <xacro:property name="wheel_radius" value="0.1"/>
     <xacro:property name="wheel_height" value="0.05"/>
-    <material name="green">
-        <color rgba = "0 1 0 1"/>
-    </material>
-    <material name="grey">
-        <color rgba = "0.5 0.5 0.5 1"/>
-    </material>
     <xacro:macro name="wheel_link" params="side color">
         <link name="${side}_wheel_link">

Commit message: feat: Inertia properties addition

File: src/MineMapper_bringup/URDF/MineMapper.urdf.xacro (robot description, xacro)
@@ -18,4 +18,6 @@
                 <material name="${color}"/>
             </visual>
+            <xacro:cylinder_inertia m = "1.0" r="${wheel_radius}" h="${wheel_height}"
+                                    xyz="0 0 0" rpy="0 0 0"/>
         </link>
     </xacro:macro>
@@ -43,4 +45,6 @@
             <material name = "green"/>
         </visual>
+        <xacro:box_inertia m = "1.0" l="${base_length}" w="${base_width}" h="${base_height}"
+                                    xyz="0 0 ${base_height/2}" rpy="0 0 0"/>
     </link>
     <xacro:wheel_link side="right" color="grey"/>
@@ -56,4 +60,6 @@
             <material name = "grey"/>
         </visual>
+        <xacro:sphere_inertia   m="1.0" r="${wheel_radius/2}"
+                                xyz="0 0 0" rpy="0 0 0"/>
     </link>
     <joint name="base_caster_wheel_joint" type="fixed">

File: src/MineMapper_bringup/URDF/commom_properties.xacro (robot description, xacro)
@@ -7,3 +7,30 @@
         <color rgba = "0.5 0.5 0.5 1"/>
     </material>
+     <xacro:macro name="box_inertia" params="m l w h xyz rpy">
+        <inertial>
+            <origin xyz="${xyz}" rpy="${rpy}"/>
+            <mass value="${m}"/>
+            <inertia    ixx="${(m/12.0)*(w*w+h*h)}" ixy="0.0" ixz="0.0"
+                        iyy="${(m/12.0)*(l*l+h*h)}" iyz="0.0"
+                        izz="${(m/12.0)*(l*l+w*w)}"/>
+        </inertial>
+    </xacro:macro>
+    <xacro:macro name="cylinder_inertia" params="m r h xyz rpy">
+        <inertial>
+            <origin xyz="${xyz}" rpy="${rpy}"/>
+            <mass value="${m}"/>
+            <inertia ixx="${(m/12.0)*(3*r*r+h*h)}" ixy="0.0" ixz="0.0"
+                    iyy="${(m/12.0)*(3*r*r+h*h)}" iyz="0.0"
+                    izz="${(m/2.0)*(r*r)}"/>
+        </inertial>
+    </xacro:macro>
+    <xacro:macro name="sphere_inertia" params="m r xyz rpy">
+        <inertial>
+            <origin xyz="${xyz}" rpy="${rpy}"/>
+            <mass value="${m}"/>
+            <inertia ixx="${(2.0*m/5.0)*(r*r)}" ixy="0.0" ixz="0.0"
+                    iyy="${(2.0*m/5.0)*(r*r)}" iyz="0.0"
+                    izz="${(2.0*m/5.0)*(r*r)}"/>
+        </inertial>
+    </xacro:macro>
 </robot>

Commit message: feat: collision addition

File: src/MineMapper_bringup/URDF/MineMapper.urdf.xacro (robot description, xacro)
@@ -18,4 +18,10 @@
                 <material name="${color}"/>
             </visual>
+            <collision>
+                <geometry>
+                    <sphere radius="${wheel_radius}"/>
+                </geometry>
+                <origin xyz="0 0 0" rpy="0 0 0"/>
+            </collision>
             <xacro:cylinder_inertia m = "1.0" r="${wheel_radius}" h="${wheel_height}"
                                     xyz="0 0 0" rpy="0 0 0"/>
@@ -45,4 +51,12 @@
             <material name = "green"/>
         </visual>
+        <collision>
+            <geometry>
+                <box size=" ${base_length}
+                            ${base_width}
+                            ${base_height}"/>
+            </geometry>
+            <origin xyz="0 0 ${base_height/2}" rpy="0 0 0"/>
+        </collision>
         <xacro:box_inertia m = "1.0" l="${base_length}" w="${base_width}" h="${base_height}"
                                     xyz="0 0 ${base_height/2}" rpy="0 0 0"/>
@@ -60,4 +74,11 @@
             <material name = "grey"/>
         </visual>
+        <collision>
+            <geometry>
+                <sphere radius="${wheel_radius/2}"/>
+            </geometry>
+            <origin xyz="0 0 0" rpy="0 0 0"/>
+            <material name = "grey"/>
+        </collision>
         <xacro:sphere_inertia   m="1.0" r="${wheel_radius/2}"
                                 xyz="0 0 0" rpy="0 0 0"/>
