Commit message: feat: gazebo implementation

File: src/MineMapper_description/URDF/MineMapper.urdf.xacro (robot description, xacro)
@@ -3,10 +3,6 @@
     <!-- INCLUDES -->
     <xacro:include filename="commom_properties.xacro"/>
-    <!-- PROPERTIES -->
-    <xacro:property name="base_length" value="0.6"/>
-    <xacro:property name="base_width" value="0.4"/>
-    <xacro:property name="base_height" value="0.2"/>
-    <xacro:property name="wheel_radius" value="0.1"/>
-    <xacro:property name="wheel_height" value="0.05"/>
+    <xacro:include filename="mobile_base_gazebo.xacro"/>
+    <xacro:include filename="dimensions.xacro"/>
     <xacro:macro name="wheel_link" params="side color">
         <link name="${side}_wheel_link">
@@ -41,4 +37,10 @@
         </joint>
     </xacro:macro>
+    <link name="base_footprint"/>
+    <joint name="base_joint" type="fixed">
+        <parent link="base_footprint"/>
+        <child link="base_link"/>
+        <origin xyz = "0 0 0" rpy = "0 0 0"/>
+    </joint>
     <link name="base_link">
         <visual>
@@ -76,10 +78,10 @@
         <collision>
             <geometry>
-                <sphere radius="${wheel_radius/2}"/>
+                <sphere radius="${caster_wheel_radius}"/>
             </geometry>
             <origin xyz="0 0 0" rpy="0 0 0"/>
             <material name = "grey"/>
         </collision>
-        <xacro:sphere_inertia   m="1.0" r="${wheel_radius/2}"
+        <xacro:sphere_inertia   m="1.0" r="${caster_wheel_radius}"
                                 xyz="0 0 0" rpy="0 0 0"/>
     </link>
@@ -87,5 +89,5 @@
         <parent link="base_link"/>
         <child link="caster_wheel"/>
-        <origin xyz = "${base_length/3} 0 ${-wheel_radius/2}" rpy = "0 0 0"/>
+        <origin xyz = "${base_length/3} 0 ${-caster_wheel_radius}" rpy = "0 0 0"/>
     </joint>
 </robot>
